File: pcb/mswi/main.sch (KiCad schematic (older format))
At the start: 4 parts

Commit message: Schematics Annotated
Connections:
- no-connect marks 1 -> 0
Changed lines of the file:
@@
 Wire Wire Line
 	6600 3300 6400 3300
-$Sheet
-S 6600 3100 1050 500
-U 5AACFFEF
-F0 "POWER SUPPLY" 60
-F1 "supplies.sch" 60
-F2 "+5V_OUT" O L 6600 3300 60
-F3 "+18V_IN" I R 7650 3300 60
-F4 "GND_IN" I R 7650 3400 50
-F5 "GND_OUT" O L 6600 3400 50
-F6 "+18V_OUT" I L 6600 3200 50
-$EndSheet
 Wire Wire Line
 	6400 3300 6400 3200
@@
 	6300 3300 4000 3300
 Connection ~ 6500 3400
-NoConn ~ 6600 3200
 Wire Wire Line
 	4550 3700 4000 3700
+$Sheet
+S 6600 3100 1050 500
+U 5AACFFEF
+F0 "POWER SUPPLY" 60
+F1 "supplies.sch" 60
+F2 "+5V_OUT" O L 6600 3300 60
+F3 "+18V_IN" I R 7650 3300 60
+F4 "GND_IN" I R 7650 3400 50
+F5 "GND_OUT" O L 6600 3400 50
+$EndSheet
 $EndSCHEMATC
