File: pcb/mswi/mswi.kicad_pcb (KiCad board)
At the start: 2 copper layers, 140 x 72.3 mm, 164 parts, among them J301 AVR-ISP-6, J302 USART, J303 I2C, J501 RJ45, Q301 BC856, Q401 BC856, Q402 BC856, Q403 BC856, Q404 BC856, Q405 BC856, Q406 BC856, Q407 BC856, Q408 BC856, Q409 BC856, Q410 BC856, Q411 BC856, Q412 BC856, Q413 BC856, Q414 BC856, Q415 BC856, Q416 BC856, Q417 BC856, Q418 BC856, Q419 BC856, Q420 BC856, Q601 si2308cds, SW401 SW_Push, SW402 SW_Push, SW403 SW_Push, SW404 SW_Push, SW405 SW_Push, SW406 SW_Push, SW407 SW_Push, SW408 SW_Push, SW409 SW_Push, SW410 SW_Push, U201 MCP2551-I/SN, U202 MCP2515-xSO, U301 ATmega328PB-AU, U601 LM7805, Y201 16MHz, Y301 16MHz

Commit message: ISP connector changed to vertical
Parts:
- J301: footprint Connector_IDC:IDC-Header_2x03_P2.54mm_Horizontal -> Connector_IDC:IDC-Header_2x03_P2.54mm_Vertical
Other:
- board text added: "TODO: [x] ISP: Change to VERTICAL Version [_] OLED: Footprint & 3D [_] SW: 3D [_] RJ45: 3D [_] Fuse: 3D [x] PCB Geometry [_] Add zenitesolar and designer identification [_] Add opensource hardware symbol"
- board text removed: "TODO: [_] ISP: Change to Horizontal Version [_] OLED: Footprint & 3D [_] SW: 3D [_] RJ45: 3D [_] Fuse: 3D [x] PCB Geometry [_] Add zenitesolar and designer identification [_] Add opensource hardware symbol"
Changed lines of the file:
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@@
     (add_net "Net-(U202-Pad6)")
   )
+  (module Connector_IDC:IDC-Header_2x03_P2.54mm_Vertical (layer F.Cu)
+    (at 88.329 -90.051)
+    (descr "Through hole straight IDC box header, 2x03, 2.54mm pitch, double rows")
+    (tags "Through hole IDC box header THT 2x03 2.54mm double row")
+    (fp_text reference J301 (at 6.105 -6.35) (layer F.SilkS)
+      (effects (font (size 1 1) (thickness 0.15)))
+    )
+    (fp_text value AVR-ISP-6 (at 6.105 11.43 180) (layer F.Fab)
+      (effects (font (size 1 1) (thickness 0.15)))
+    )
+    (fp_line (start -3.655 -5.6) (end -1.115 -5.6) (layer F.SilkS) (width 0.12))
+    (fp_line (start -3.655 -5.6) (end -3.655 -3.06) (layer F.SilkS) (width 0.12))
+    (fp_line (start -3.405 -5.35) (end 5.945 -5.35) (layer F.SilkS) (width 0.12))
+    (fp_line (start -3.405 10.43) (end -3.405 -5.35) (layer F.SilkS) (width 0.12))
+    (fp_line (start 5.945 10.43) (end -3.405 10.43) (layer F.SilkS) (width 0.12))
+    (fp_line (start 5.945 -5.35) (end 5.945 10.43) (layer F.SilkS) (width 0.12))
+    (fp_line (start -3.41 -5.35) (end 5.95 -5.35) (layer F.CrtYd) (width 0.05))
+    (fp_line (start -3.41 10.43) (end -3.41 -5.35) (layer F.CrtYd) (width 0.05))
+    (fp_line (start 5.95 10.43) (end -3.41 10.43) (layer F.CrtYd) (width 0.05))
+    (fp_line (start 5.95 -5.35) (end 5.95 10.43) (layer F.CrtYd) (width 0.05))
+    (fp_line (start -3.155 10.18) (end -2.605 9.62) (layer F.Fab) (width 0.1))
+    (fp_line (start -3.155 -5.1) (end -2.605 -4.56) (layer F.Fab) (width 0.1))
+    (fp_line (start 5.695 10.18) (end 5.145 9.62) (layer F.Fab) (width 0.1))
+    (fp_line (start 5.695 -5.1) (end 5.145 -4.56) (layer F.Fab) (width 0.1))
+    (fp_line (start 5.145 9.62) (end -2.605 9.62) (layer F.Fab) (width 0.1))
+    (fp_line (start 5.695 10.18) (end -3.155 10.18) (layer F.Fab) (width 0.1))
+    (fp_line (start 5.145 -4.56) (end -2.605 -4.56) (layer F.Fab) (width 0.1))
+    (fp_line (start 5.695 -5.1) (end -3.155 -5.1) (layer F.Fab) (width 0.1))
+    (fp_line (start -2.605 4.79) (end -3.155 4.79) (layer F.Fab) (width 0.1))
+    (fp_line (start -2.605 0.29) (end -3.155 0.29) (layer F.Fab) (width 0.1))
+    (fp_line (start -2.605 4.79) (end -2.605 9.62) (layer F.Fab) (width 0.1))
+    (fp_line (start -2.605 -4.56) (end -2.605 0.29) (layer F.Fab) (width 0.1))
+    (fp_line (start -3.155 -5.1) (end -3.155 10.18) (layer F.Fab) (width 0.1))
+    (fp_line (start 5.145 -4.56) (end 5.145 9.62) (layer F.Fab) (width 0.1))
+    (fp_line (start 5.695 -5.1) (end 5.695 10.18) (layer F.Fab) (width 0.1))
+    (fp_text user %R (at 8.805 2.54 90) (layer F.Fab)
+      (effects (font (size 1 1) (thickness 0.15)))
+    )
+    (pad 6 thru_hole oval (at 2.54 5.08) (size 1.7272 1.7272) (drill 1.016) (layers *.Cu *.Mask)
+      (net 1 GND))
+    (pad 5 thru_hole oval (at 0 5.08) (size 1.7272 1.7272) (drill 1.016) (layers *.Cu *.Mask)
+      (net 59 "Net-(J301-Pad5)"))
+    (pad 4 thru_hole oval (at 2.54 2.54) (size 1.7272 1.7272) (drill 1.016) (layers *.Cu *.Mask)
+      (net 60 "Net-(J301-Pad4)"))
+    (pad 3 thru_hole oval (at 0 2.54) (size 1.7272 1.7272) (drill 1.016) (layers *.Cu *.Mask)
+      (net 61 "Net-(J301-Pad3)"))
+    (pad 2 thru_hole oval (at 2.54 0) (size 1.7272 1.7272) (drill 1.016) (layers *.Cu *.Mask)
+      (net 2 +5V))
+    (pad 1 thru_hole rect (at 0 0) (size 1.7272 1.7272) (drill 1.016) (layers *.Cu *.Mask)
+      (net 62 "Net-(J301-Pad1)"))
+    (model ${KISYS3DMOD}/Connector_IDC.3dshapes/IDC-Header_2x03_P2.54mm_Vertical.wrl
+      (at (xyz 0 0 0))
+      (scale (xyz 1 1 1))
+      (rotate (xyz 0 0 0))
+    )
+  )
   (module Crystal:Crystal_HC49-U_Vertical (layer F.Cu)
     (at 106.394 -92.636)
@@
     )
   )
-  (module Connector_IDC:IDC-Header_2x03_P2.54mm_Horizontal (layer F.Cu)
-    (at 88.329 -90.051)
-    (descr "Through hole angled IDC box header, 2x03, 2.54mm pitch, double rows")
-    (tags "Through hole IDC box header THT 2x03 2.54mm double row")
-    (fp_text reference J301 (at 6.105 -6.35) (layer F.SilkS)
-      (effects (font (size 1 1) (thickness 0.15)))
-    )
-    (fp_text value AVR-ISP-6 (at 6.105 11.43 180) (layer F.Fab)
-      (effects (font (size 1 1) (thickness 0.15)))
-    )
-    (fp_line (start 13.48 10.43) (end -1.12 10.43) (layer F.CrtYd) (width 0.05))
-    (fp_line (start 13.48 -5.35) (end 13.48 10.43) (layer F.CrtYd) (width 0.05))
-    (fp_line (start -1.12 10.43) (end -1.12 -5.35) (layer F.CrtYd) (width 0.05))
-    (fp_line (start -1.12 -5.35) (end 13.48 -5.35) (layer F.CrtYd) (width 0.05))
-    (fp_line (start 4.13 4.79) (end 13.48 4.79) (layer F.SilkS) (width 0.12))
-    (fp_line (start 4.13 10.43) (end 4.13 -5.35) (layer F.SilkS) (width 0.12))
-    (fp_line (start 4.13 10.43) (end 13.48 10.43) (layer F.SilkS) (width 0.12))
-    (fp_line (start 4.13 0.29) (end 13.48 0.29) (layer F.SilkS) (width 0.12))
-    (fp_line (start 4.13 -5.35) (end 13.48 -5.35) (layer F.SilkS) (width 0.12))
-    (fp_line (start 13.48 -5.35) (end 13.48 10.43) (layer F.SilkS) (width 0.12))
-    (fp_line (start 0 -1.27) (end -1.27 -1.27) (layer F.SilkS) (width 0.12))
-    (fp_line (start -1.27 -1.27) (end -1.27 0) (layer F.SilkS) (width 0.12))
-    (fp_line (start 5.38 -5.1) (end 13.23 -5.1) (layer F.Fab) (width 0.1))
-    (fp_line (start 4.38 4.79) (end 13.23 4.79) (layer F.Fab) (width 0.1))
-    (fp_line (start 4.38 4.76) (end -0.32 4.76) (layer F.Fab) (width 0.1))
-    (fp_line (start 4.38 2.22) (end -0.32 2.22) (layer F.Fab) (width 0.1))
-    (fp_line (start 4.38 10.18) (end 4.38 -4.1) (layer F.Fab) (width 0.1))
-    (fp_line (start 4.38 10.18) (end 13.23 10.18) (layer F.Fab) (width 0.1))
-    (fp_line (start 4.38 0.29) (end 13.23 0.29) (layer F.Fab) (width 0.1))
-    (fp_line (start 4.38 -4.1) (end 5.38 -5.1) (layer F.Fab) (width 0.1))
-    (fp_line (start 4.38 -0.32) (end -0.32 -0.32) (layer F.Fab) (width 0.1))
-    (fp_line (start 13.23 10.18) (end 13.23 -5.1) (layer F.Fab) (width 0.1))
-    (fp_line (start -0.32 5.4) (end 4.38 5.4) (layer F.Fab) (width 0.1))
-    (fp_line (start -0.32 4.76) (end -0.32 5.4) (layer F.Fab) (width 0.1))
-    (fp_line (start -0.32 2.86) (end 4.38 2.86) (layer F.Fab) (width 0.1))
-    (fp_line (start -0.32 2.22) (end -0.32 2.86) (layer F.Fab) (width 0.1))
-    (fp_line (start -0.32 0.32) (end 4.38 0.32) (layer F.Fab) (width 0.1))
-    (fp_line (start -0.32 -0.32) (end -0.32 0.32) (layer F.Fab) (width 0.1))
-    (fp_text user %R (at 8.805 2.54 90) (layer F.Fab)
-      (effects (font (size 1 1) (thickness 0.15)))
-    )
-    (pad 6 thru_hole oval (at 2.54 5.08) (size 1.7272 1.7272) (drill 1.016) (layers *.Cu *.Mask)
-      (net 1 GND))
-    (pad 5 thru_hole oval (at 0 5.08) (size 1.7272 1.7272) (drill 1.016) (layers *.Cu *.Mask)
-      (net 59 "Net-(J301-Pad5)"))
-    (pad 4 thru_hole oval (at 2.54 2.54) (size 1.7272 1.7272) (drill 1.016) (layers *.Cu *.Mask)
-      (net 60 "Net-(J301-Pad4)"))
-    (pad 3 thru_hole oval (at 0 2.54) (size 1.7272 1.7272) (drill 1.016) (layers *.Cu *.Mask)
-      (net 61 "Net-(J301-Pad3)"))
-    (pad 2 thru_hole oval (at 2.54 0) (size 1.7272 1.7272) (drill 1.016) (layers *.Cu *.Mask)
-      (net 2 +5V))
-    (pad 1 thru_hole rect (at 0 0) (size 1.7272 1.7272) (drill 1.016) (layers *.Cu *.Mask)
-      (net 62 "Net-(J301-Pad1)"))
-    (model ${KISYS3DMOD}/Connector_IDC.3dshapes/IDC-Header_2x03_P2.54mm_Horizontal.wrl
-      (at (xyz 0 0 0))
-      (scale (xyz 1 1 1))
-      (rotate (xyz 0 0 0))
-    )
-  )
   (module MountingHole:MountingHole_3.2mm_M3 (layer F.Cu)
     (at 90.474 -58.036)
@@
   (gr_line (start 265.355981 50.910094) (end 265.355981 123.214313) (layer Dwgs.User) (width 0.4))
   (gr_line (start 163.461214 123.214313) (end 267.355981 123.214313) (layer Dwgs.User) (width 0.4))
-  (gr_text "TODO:\n[_] ISP: Change to Horizontal Version\n[_] OLED: Footprint & 3D\n[_] SW: 3D\n[_] RJ45: 3D\n[_] Fuse: 3D\n[x] PCB Geometry \n[_] Add zenitesolar and designer identification\n[_] Add opensource hardware symbol\n" (at 125 180) (layer Eco2.User)
+  (gr_text "TODO:\n[x] ISP: Change to VERTICAL Version\n[_] OLED: Footprint & 3D\n[_] SW: 3D\n[_] RJ45: 3D\n[_] Fuse: 3D\n[x] PCB Geometry \n[_] Add zenitesolar and designer identification\n[_] Add opensource hardware symbol\n" (at 125 180) (layer Eco2.User)
     (effects (font (size 1.5 1.5) (thickness 0.1)) (justify left))
   )
