File: pcb/mswi/mswi.kicad_pcb (KiCad board)
At the start: 2 copper layers, 140 x 72.3 mm, 166 parts, among them J301 AVR-ISP-6, J302 USART, J303 I2C, J501 Conn_01x04_Male, Q301 BC856, Q401 BC856, Q402 BC856, Q403 BC856, Q404 BC856, Q405 BC856, Q406 BC856, Q407 BC856, Q408 BC856, Q409 BC856, Q410 BC856, Q411 BC856, Q412 BC856, Q413 BC856, Q414 BC856, Q415 BC856, Q416 BC856, Q417 BC856, Q418 BC856, Q419 BC856, Q420 BC856, Q601 si2308cds, SW401 SW_Push, SW402 SW_Push, SW403 SW_Push, SW404 SW_Push, SW405 SW_Push, SW406 SW_Push, SW407 SW_Push, SW408 SW_Push, SW409 SW_Push, SW410 SW_Push, U201 MCP2551-I/SN, U202 MCP2515-xSO, U301 ATmega328PB-AU, U601 LM7805, Y201 16MHz, Y301 16MHz

Commit message: working...
Parts:
- removed H101, H102, H103, H104: MountingHole, MountingHole:MountingHole_3.2mm_M3
- C301, Y201, Y301: moved to B.Cu
- moved BZ301 85.1 mm to (228.0, -73.4)
- moved D306 85.1 mm to (234.0, -65.7)
- moved Q301 85.1 mm to (233.2, -69.9)
- moved R318 85.1 mm to (234.0, -76.9)
- moved R319 85.1 mm to (231.5, -73.9)
- moved R320 85.1 mm to (237.8, -66.7)
- moved TP306 85.1 mm to (229.5, -77.2)
- moved TP307 85.1 mm to (229.0, -69.2)
- moved U301 65.1 mm to (220.8, -32.4), turned to 45 degrees
- moved Y301 56.9 mm to (206.0, -20.6), turned to 90 degrees
- moved C301 51.8 mm to (216.8, -28.6), turned to 315 degrees
- moved C605 41.9 mm to (91.6, -24.4)
- moved Q601 41.9 mm to (102.8, -32.4)
- moved R601 41.9 mm to (97.8, -33.4)
- moved U601 41.9 mm to (85.8, -32.4)
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Routing:
- net +5V: track 27.2 -> 70.4 mm, vias 2 -> 5
- net GND: track 415.9 -> 453.0 mm, vias 12 -> 16
- net /CANBUS/TXCAN: track 0.00 -> 12.7 mm
- net /CANBUS/RXCAN: track 0.00 -> 11.3 mm
- net Net-(C203-Pad1): track 0.00 -> 8.42 mm
- net Net-(C306-Pad1): track 0.00 -> 6.34 mm
- net Net-(C204-Pad1): track 0.00 -> 5.74 mm
- net Net-(C305-Pad1): track 0.00 -> 5.00 mm
- net Net-(R203-Pad2): track 0.00 -> 4.47 mm
- net /CANBUS CONN/CAN_L: track 0.00 -> 3.69 mm
- net /CANBUS CONN/CAN_H: track 0.00 -> 3.69 mm
- net /MCU/LED0: track 0.00 -> 3.25 mm
- net /MCU/LED1: track 0.00 -> 2.86 mm
- net Net-(R202-Pad1): track 0.00 -> 2.50 mm
- net /MCU/SW2: track 20.1 -> 22.2 mm
Other:
- net class Default: clearance 0.508 -> 0.127; trace_width 0.508 -> 0.381
- rule trace_clearance: 0.508 -> 0.127

Commit message: routing: wip
Parts:
- removed TP201: SI, TestPoint:TestPoint_Pad_2.0x2.0mm
- removed TP202: SO, TestPoint:TestPoint_Pad_2.0x2.0mm
- removed TP205: SC, TestPoint:TestPoint_Pad_2.0x2.0mm
- removed TP206: SCK, TestPoint:TestPoint_Pad_2.0x2.0mm
- removed TP209: INT, TestPoint:TestPoint_Pad_2.0x2.0mm
- removed TP301: TX, TestPoint:TestPoint_Pad_2.0x2.0mm
- removed TP302: RX, TestPoint:TestPoint_Pad_2.0x2.0mm
- removed TP303: RST, TestPoint:TestPoint_Pad_2.0x2.0mm
- removed TP304: SDA, TestPoint:TestPoint_Pad_2.0x2.0mm
- removed TP305: SCL, TestPoint:TestPoint_Pad_2.0x2.0mm
- added C602: 100nF, Capacitor_SMD:C_0805_2012Metric_Pad1.15x1.40mm_HandSolder, B.Cu at (99.4, 150.0)
- C302, C303, C304, C307, C308, D201, D301, L301, R201, R301, R302, R303, R304, R311, R312, R313, SW403, SW404, SW407, SW408, TP207, TP208: moved to B.Cu
- C403, C404, C407, C408, Q403, Q404, Q408, Q409, Q412, Q413, Q417, Q418, R403, R404, R408, R409, R413, R414, R417, R418, R422, R423, R427, R428: moved to F.Cu
- J301: value AVR-ISP-6 -> ISP; footprint Connector_IDC:IDC-Header_2x03_P2.54mm_Vertical -> Connector_PinHeader_2.54mm:PinHeader_1x06_P2.54mm_Vertical
- moved R403 314.2 mm to (104.3, 60.8), turned to 228.2 degrees
- moved Q403 311.2 mm to (103.9, 66.2), turned to 228.2 degrees
- moved Q408 308.4 mm to (106.5, 63.2), turned to 228.2 degrees
- moved SW403 306.4 mm to (104.2, 72.2), turned to 48.2 degrees
- moved R408 302.3 mm to (107.1, 70.4), turned to 318.2 degrees
- moved C403 301.0 mm to (109.3, 66.6), turned to 48.2 degrees
- moved D403 299.0 mm to (113.4, 58.6), turned to 318.2 degrees
- moved R413 296.5 mm to (111.1, 68.3), turned to 228.2 degrees
- moved R418 287.5 mm to (115.2, 70.5), turned to 228.2 degrees
- moved Q413 284.5 mm to (114.7, 75.9), turned to 228.2 degrees
- moved Q418 281.7 mm to (117.4, 72.9), turned to 228.2 degrees
- moved SW408 279.7 mm to (115.1, 81.9), turned to 48.2 degrees
- moved R417 277.8 mm to (167.3, 78.1), turned to 311.8 degrees
- moved SW410 275.9 mm to (102.3, 97.2), turned to 48.2 degrees
- moved R423 275.6 mm to (118.0, 80.1), turned to 318.2 degrees
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Connections:
- J301 pad 1: Net-(J301-Pad1) -> GND
- J301 pad 6: GND -> Net-(J301-Pad6)
- J303 pad 1: GND -> +5V
- J303 pad 2: +5V -> GND
- R301 pad 1: /CANBUS/SO -> /MCU/SPI_MOSI_
- R301 pad 2: Net-(J301-Pad1) -> Net-(J301-Pad6)
- R302 pad 1: /CANBUS/SI -> /MCU/SPI_MISO_
- R302 pad 2: Net-(J301-Pad4) -> Net-(J301-Pad5)
- R303 pad 1: /CANBUS/SCK -> /MCU/SPI_SCK_
- R303 pad 2: Net-(J301-Pad3) -> Net-(J301-Pad4)
- R304 pad 2: Net-(J301-Pad5) -> Net-(J301-Pad3)
- R305 pad 1: /CANBUS/SI -> /MCU/SPI_MOSI_
- R306 pad 1: /CANBUS/SO -> /MCU/SPI_MISO_
- R307 pad 1: /CANBUS/SCK -> /MCU/SPI_SCK_
- U301 pad 12: /CANBUS/CS -> /MCU/BUZZER
- U301 pad 13: /CANBUS/INT -> /CANBUS/CS
- U301 pad 14: /MCU/BUZZER -> /CANBUS/INT
- U301 pad 15: /CANBUS/SI -> /MCU/SPI_MOSI_
- U301 pad 16: /CANBUS/SO -> /MCU/SPI_MISO_
- U301 pad 17: /CANBUS/SCK -> /MCU/SPI_SCK_
- U601 pad : GND -> (no net)
Routing:
- net GND: track 453.0 -> 534.5 mm, vias 16 -> 19
- net +5V: track 70.4 -> 131.3 mm, vias 5 -> 7
- net /MCU/RESET: track 0.00 -> 42.8 mm, vias 0 -> 1
- net /CANBUS/CS: track 0.00 -> 29.5 mm
- net /MCU/SPI_MOSI_: track 0.00 -> 26.3 mm, vias 0 -> 1
- net /MCU/SPI_MISO_: track 0.00 -> 21.7 mm, vias 0 -> 1
- net /CANBUS/INT: track 0.00 -> 20.8 mm
- net /MCU/USART_RX: track 0.00 -> 18.8 mm
- net /MCU/SPI_SCK_: track 0.00 -> 18.3 mm, vias 0 -> 1
- net /MCU/USART_TX: track 0.00 -> 17.0 mm
- net /CANBUS/SCK: track 0.00 -> 16.2 mm, vias 0 -> 2
- net /MCU/I2C_SDA: track 0.00 -> 16.1 mm, vias 0 -> 1
- net /MCU/I2C_SCL: track 0.00 -> 15.3 mm, vias 0 -> 1
- net /CANBUS/SO: track 0.00 -> 15.3 mm
- net /CANBUS CONN/CAN_H: track 3.69 -> 18.6 mm, vias 0 -> 1
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Other:
- board text added: "TODO: [_] Adapt Rules to Fabrication Method [x] ISP: Change to VERTICAL Version [x] OLED: Footprint & 3D [_] SW: 3D [_] RJ45: 3D [_] Fuse: 3D [x] PCB Geometry [_] Add zenitesolar and designer identification [_] Add opensource hardware symbol [_] Define the switches position -> paper prototype"
- board text removed: "TODO: [_] Adapt Rules to Fabrication Method [x] ISP: Change to VERTICAL Version [_] OLED: Footprint & 3D [_] SW: 3D [_] RJ45: 3D [_] Fuse: 3D [x] PCB Geometry [_] Add zenitesolar and designer identification [_] Add opensource hardware symbol [_] Define the switches position -> paper prototype"
