File: pcb/mswi/switches.sch (KiCad schematic (older format))
At the start: 80 parts

Commit message: Schematics Annotated
Parts:
- gave numbers to parts that had none: 80

Commit message: Footprints associated
Parts:
- SW401, SW402, SW403, SW404, SW405, SW406, SW407, SW408, SW409, SW410: footprint (none) -> Button_Switch_THT:SW_PUSH-12mm
Changed lines of the file:
@@
 F 0 "SW401" V 3700 3100 50  0000 R CNN
 F 1 "SW_Push" H 3700 3300 50  0001 C CNN
-F 2 "" H 3700 3300 50  0001 C CNN
+F 2 "Button_Switch_THT:SW_PUSH-12mm" H 3700 3300 50  0001 C CNN
 F 3 "~" H 3700 3300 50  0001 C CNN
 	1    3700 3100
@@
 F 0 "SW402" V 4800 3100 50  0000 R CNN
 F 1 "SW_Push" H 4800 3300 50  0001 C CNN
-F 2 "" H 4800 3300 50  0001 C CNN
+F 2 "Button_Switch_THT:SW_PUSH-12mm" H 4800 3300 50  0001 C CNN
 F 3 "~" H 4800 3300 50  0001 C CNN
 	1    4800 3100
@@
 F 0 "SW403" V 5900 3100 50  0000 R CNN
 F 1 "SW_Push" H 5900 3300 50  0001 C CNN
-F 2 "" H 5900 3300 50  0001 C CNN
+F 2 "Button_Switch_THT:SW_PUSH-12mm" H 5900 3300 50  0001 C CNN
 F 3 "~" H 5900 3300 50  0001 C CNN
 	1    5900 3100
@@
 F 0 "SW404" V 7000 3100 50  0000 R CNN
 F 1 "SW_Push" H 7000 3300 50  0001 C CNN
-F 2 "" H 7000 3300 50  0001 C CNN
+F 2 "Button_Switch_THT:SW_PUSH-12mm" H 7000 3300 50  0001 C CNN
 F 3 "~" H 7000 3300 50  0001 C CNN
 	1    7000 3100
@@
 F 0 "SW405" V 8100 3150 50  0000 R CNN
 F 1 "SW_Push" H 8100 3350 50  0001 C CNN
-F 2 "" H 8100 3350 50  0001 C CNN
+F 2 "Button_Switch_THT:SW_PUSH-12mm" H 8100 3350 50  0001 C CNN
 F 3 "~" H 8100 3350 50  0001 C CNN
 	1    8100 3150
@@
 F 0 "SW406" V 3700 5300 50  0000 R CNN
 F 1 "SW_Push" H 3700 5500 50  0001 C CNN
-F 2 "" H 3700 5500 50  0001 C CNN
+F 2 "Button_Switch_THT:SW_PUSH-12mm" H 3700 5500 50  0001 C CNN
 F 3 "~" H 3700 5500 50  0001 C CNN
 	1    3700 5300
@@
 F 0 "SW407" V 4800 5300 50  0000 R CNN
 F 1 "SW_Push" H 4800 5500 50  0001 C CNN
-F 2 "" H 4800 5500 50  0001 C CNN
+F 2 "Button_Switch_THT:SW_PUSH-12mm" H 4800 5500 50  0001 C CNN
 F 3 "~" H 4800 5500 50  0001 C CNN
 	1    4800 5300
@@
 F 0 "SW408" V 5900 5300 50  0000 R CNN
 F 1 "SW_Push" H 5900 5500 50  0001 C CNN
-F 2 "" H 5900 5500 50  0001 C CNN
+F 2 "Button_Switch_THT:SW_PUSH-12mm" H 5900 5500 50  0001 C CNN
 F 3 "~" H 5900 5500 50  0001 C CNN
 	1    5900 5300
@@
 F 0 "SW409" V 7000 5300 50  0000 R CNN
 F 1 "SW_Push" H 7000 5500 50  0001 C CNN
-F 2 "" H 7000 5500 50  0001 C CNN
+F 2 "Button_Switch_THT:SW_PUSH-12mm" H 7000 5500 50  0001 C CNN
 F 3 "~" H 7000 5500 50  0001 C CNN
 	1    7000 5300
@@
 F 0 "SW410" V 8100 5350 50  0000 R CNN
 F 1 "SW_Push" H 8100 5550 50  0001 C CNN
-F 2 "" H 8100 5550 50  0001 C CNN
+F 2 "Button_Switch_THT:SW_PUSH-12mm" H 8100 5550 50  0001 C CNN
 F 3 "~" H 8100 5550 50  0001 C CNN
 	1    8100 5350
